File: hardware/BioAmpShield.kicad_sch (KiCad schematic)
At the start: 50 parts, among them U2 opamp

Commit message: Update hardware
Parts:
- C1: value (none) -> 47uF; footprint (none) -> Capacitor_THT:CP_Radial_D5.0mm_P2.50mm
- C10, C2, C3, C9: value (none) -> CP; footprint (none) -> Capacitor_THT:CP_Radial_D5.0mm_P2.50mm
- C4: value (none) -> 20nF; footprint (none) -> Capacitor_THT:C_Disc_D3.8mm_W2.6mm_P2.50mm
- C5: value (none) -> 100nF; footprint (none) -> Capacitor_THT:C_Disc_D3.8mm_W2.6mm_P2.50mm
- C6: value (none) -> 47nF; footprint (none) -> Capacitor_THT:C_Disc_D3.8mm_W2.6mm_P2.50mm
- C7, C8: value (none) -> 220nF; footprint (none) -> Capacitor_THT:C_Disc_D3.8mm_W2.6mm_P2.50mm
- D1: value (none) -> D; footprint (none) -> Diode_THT:D_DO-35_SOD27_P7.62mm_Horizontal
- D2, D3, D4, D5, D6, D7, D8: value (none) -> LED; footprint (none) -> LED_THT:LED_D5.0mm
- J1: value (none) -> Conn_01x03; footprint (none) -> Connector_PinHeader_2.54mm:PinHeader_1x03_P2.54mm_Vertical
- J2: value (none) -> SJ1-3525N; footprint (none) -> udlabs:CUI_SJ1-3525N
- J3: value (none) -> Conn_01x03; footprint (none) -> Connector_JST:JST_PH_S3B-PH-K_1x03_P2.00mm_Horizontal
- J4: value (none) -> Conn_01x02; footprint (none) -> Connector_JST:JST_PH_S2B-PH-K_1x02_P2.00mm_Horizontal
- P1: value (none) -> Power; footprint (none) -> Socket_Arduino_Uno:Socket_Strip_Arduino_1x08
- P2: value (none) -> Analog; footprint (none) -> Socket_Arduino_Uno:Socket_Strip_Arduino_1x06
- P3: value (none) -> Digital; footprint (none) -> Socket_Arduino_Uno:Socket_Strip_Arduino_1x10
- P4: value (none) -> Digital; footprint (none) -> Socket_Arduino_Uno:Socket_Strip_Arduino_1x08
- R1: value (none) -> 10k; footprint (none) -> Resistor_THT:R_Axial_DIN0207_L6.3mm_D2.5mm_P2.54mm_Vertical
- R10, R11, R12, R13, R14, R15, R16, R2, R20, R4, R7, R8: value (none) -> 1K; footprint (none) -> Resistor_THT:R_Axial_DIN0207_L6.3mm_D2.5mm_P2.54mm_Vertical
- R17, R18, R19, R9: value (none) -> 1M; footprint (none) -> Resistor_THT:R_Axial_DIN0207_L6.3mm_D2.5mm_P2.54mm_Vertical
- R3: value (none) -> 100k; footprint (none) -> Resistor_THT:R_Axial_DIN0207_L6.3mm_D2.5mm_P2.54mm_Vertical
- R5, R6: value (none) -> 10K; footprint (none) -> Resistor_THT:R_Axial_DIN0207_L6.3mm_D2.5mm_P2.54mm_Vertical
- RV1: value (none) -> R_POT_Small; footprint (none) -> Potentiometer_THT:Potentiometer_Runtron_RM-065_Vertical
- SW1, SW2: value (none) -> SW_Push; footprint (none) -> Button_Switch_THT:SW_PUSH_6mm_H5mm
- U2: value opamp -> TL074; footprint (none) -> Package_DIP:DIP-14_W7.62mm_Socket_LongPads
Other:
- company: Upside Down Labs -> (none)
- title: Muscle BioAmp Shield -> (none)

Commit message: Update final design
Other:
- company: (none) -> Upside Down Labs
- title: (none) -> Muscle BioAmp Shield
