File: hardware/Muscle-BioAmpShield.kicad_pcb (KiCad board)
At the start: 2 copper layers, 52.1 x 53.3 mm, 53 parts, among them J1 Audio_output, J2 BioAmp_input, J3 Board_power, J4 Digital_pins, J5 PJ-3062-CO, P1 Power, P2 Analog, P3 Digital, P4 Digital, SW1 SW_Push, SW2 SW_Push, U1 Amp

Commit message: Update to v0.3 KiCad files
Parts:
- removed the C12 at (138.7, 113.3)
- removed LOGO1: LOGO_UDLABS, udlabs:upsidedownlabsLOGO_41x34
- removed the R3 at (149.2, 102.3)
- removed the R6 at (149.2, 96.3)
- added C11: 100nF, Capacitor_THT:C_Disc_D3.8mm_W2.6mm_P2.50mm, F.Cu at (131.8, 112.9)
- added G***: LOGO, UDLEOG:CandyMuscle, B.Cu at (158.5, 99.4)
- added J10: Servo motor, Connector_PinHeader_2.54mm:PinHeader_1x03_P2.54mm_Vertical, F.Cu at (171.4, 77.7)
- added J6: Isolated Output, Connector_JST:JST_PH_B2B-PH-K_1x02_P2.00mm_Vertical, F.Cu at (161.0, 89.6)
- added J7: Stemma Analog A2, Connector_JST:JST_PH_B3B-PH-K_1x03_P2.00mm_Vertical, F.Cu at (148.9, 116.8)
- added J8: Stemma I2C, Connector_JST:JST_PH_S4B-PH-K_1x04_P2.00mm_Horizontal, F.Cu at (122.5, 74.8)
- added J9: Battery Power, Connector_JST:JST_PH_S2B-PH-K_1x02_P2.00mm_Horizontal, F.Cu at (126.8, 118.4)
- added U2: PC817, Package_DIP:DIP-4_W7.62mm, F.Cu at (166.2, 77.0)
- added kibuzzard-63B5E73F: G***, kibuzzard-63B5E73F, F.Cu at (153.2, 105.3)
- added kibuzzard-63B65023: G***, kibuzzard-63B65023, B.Cu at (147.2, 97.7)
- added kibuzzard-63B67C69: G***, kibuzzard-63B67C69, B.Cu at (122.8, 104.7)
- C1: renamed from C11; value 47uF -> 2.2uF
- C10: value 47uF -> 470uF
- C12: renamed from C6; value 10uF -> 470uF
- C3: renamed from C1; value 1nF -> 100pF
- C5: renamed from C3; value 1nF -> 100pF
- C6: renamed from C8; value 2.2uF -> 1uF
- C8: renamed from C4; value 100nF -> 100pF
- J1: renamed from J2; value BioAmp_input -> BioAmp Input
- J3: value Board_power -> Stemma I2C; footprint Connector_JST:JST_PH_S2B-PH-K_1x02_P2.00mm_Horizontal -> Connector_JST:JST_PH_B4B-PH-K_1x04_P2.00mm_Vertical
- J4: value Digital_pins -> Stemma Digital D6; footprint Connector_PinHeader_2.54mm:PinHeader_1x04_P2.54mm_Vertical -> Connector_JST:JST_PH_B3B-PH-K_1x03_P2.00mm_Vertical
- R1: renamed from R7; value 1K -> 1M
- R19: renamed from R11; value 15K -> 10K
- R2: renamed from R8; value 1K -> 1M
- R20: renamed from R12; value 15K -> 10K
- R5: renamed from R4; value 10K -> 220K
- R6: renamed from R1; value 1K -> 22K
- R7: renamed from R5; value 1K -> 22K
- R8: renamed from R2; value 10K -> 220K
- moved J4 50.7 mm to (139.9, 116.8), turned to 180 degrees
- moved J3 32.7 mm to (159.9, 116.8), turned to 180 degrees
- moved D6 12.9 mm to (120.0, 122.6), turned to 90 degrees
- moved C5 12.7 mm to (134.7, 111.9), turned to 0 degrees
- moved D5 12.5 mm to (120.0, 115.7), turned to 90 degrees
- moved C6 12.2 mm to (148.6, 110.3)
- moved D4 12.2 mm to (120.0, 108.8), turned to 90 degrees
- moved D3 11.9 mm to (120.0, 101.9), turned to 90 degrees
- moved SW1 11.8 mm to (152.9, 83.9), turned to 90 degrees
- moved D2 11.5 mm to (120.0, 95.0), turned to 90 degrees
- moved D1 11.2 mm to (120.0, 88.1), turned to 90 degrees
- moved C8 10.5 mm to (125.5, 96.4)
- moved R19 10.5 mm to (160.5, 76.9), turned to -90 degrees
- moved C2 8.78 mm to (125.5, 99.9)
- moved R6 8.32 mm to (151.0, 99.3)
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- renumbered C7 to C2, C2 to C4, C5 to C7, J5 to J2, J1 to J5, R15 to R10, R13 to R11, R16 to R12, R17 to R13, R18 to R14, R19 to R15, R20 to R16, R21 to R17, R22 to R18, R10 to R3, R9 to R4, R14 to R9
Connections:
- net /10(**/SS) renamed /10(**/SS)
- net /11(**/MOSI) renamed /11(**/MOSI)
- C10 pad 1: +5V -> 5V
- C10 pad 2: Ring2 -> GND
- C12 pad 1: ampRef -> 9V
- C12 pad 2: Ring2 -> GND
- C2 pad 1: Ring2 -> GND
- C2 pad 2: Net-(C4-Pad1) -> Net-(C2-Pad2)
- C8 pad 1: Net-(C4-Pad1) -> GND
- C8 pad 2: +5V -> ampRef
- C9 pad 1: Ring2 -> GND
- C9 pad 2: +5V -> 5V
- D1 pad 1: Ring2 -> GND
- D2 pad 1: Ring2 -> GND
- D3 pad 1: Ring2 -> GND
- D4 pad 1: Ring2 -> GND
- D5 pad 1: Ring2 -> GND
- D6 pad 1: Ring2 -> GND
- J1 pad 1: bioIN- -> inaIN-
- J1 pad 2: bioIN+ -> inaIN+
- J2 pad 1: Ring2 -> GND
- J3 pad 1: +9V -> /A5(SCL)
- J3 pad 2: Ring2 -> /A4(SDA)
- J4 pad 1: /2 -> /6(**)
- J4 pad 2: /3(**) -> 5V
- J4 pad 3: /5(**) -> GND
- J5 pad 3: Ring2 -> GND
- P1 pad 1: (no net) -> unconnected-(P1-Pad1)
- P1 pad 2: (no net) -> /IOREF
- P1 pad 3: (no net) -> /Reset
- P1 pad 4: (no net) -> +3V3
- P1 pad 5: +5V -> 5V
- P1 pad 6: Ring2 -> GND
- P1 pad 7: Ring2 -> GND
- P1 pad 8: +9V -> 9V
- P2 pad 2: (no net) -> /A1
- P2 pad 3: (no net) -> /A2
- P2 pad 4: (no net) -> /A3
- P2 pad 5: (no net) -> /A4(SDA)
- P2 pad 6: (no net) -> /A5(SCL)
- P3 pad 1: (no net) -> SCL
- P3 pad 2: (no net) -> SDA
- P3 pad 3: (no net) -> /AREF
- P3 pad 4: Ring2 -> GND
- P4 pad 2: (no net) -> /6(**)
- P4 pad 7: (no net) -> /1(Tx)
- P4 pad 8: (no net) -> /0(Rx)
- R1 pad 1: Net-(C4-Pad1) -> Net-(C2-Pad2)
- R1 pad 2: +5V -> 5V
- R12 pad 2: Ring2 -> GND
- R19 pad 1: Ring2 -> GND
- R2 pad 1: Ring2 -> GND
- R2 pad 2: Net-(C4-Pad1) -> Net-(C2-Pad2)
- R20 pad 1: Ring2 -> GND
- SW1 pad 1: +5V -> 5V
- SW2 pad 1: +5V -> 5V
- U1 pad 11: Ring2 -> GND
- U1 pad 12: Net-(C4-Pad1) -> Net-(C2-Pad2)
- U1 pad 4: +5V -> 5V
Routing:
- net Ring2: track 228.7 -> 0.00 mm
- net 5V: track 0.00 -> 213.0 mm
- net +5V: track 124.1 -> 0.00 mm
- net 9V: track 0.00 -> 74.7 mm
- net /6(**): track 0.00 -> 53.4 mm
- net GND: track 0.00 -> 38.5 mm, vias 0 -> 204
- net inaIN-: track 30.2 -> 67.6 mm
- net Net-(C6-Pad1): track 54.9 -> 22.3 mm
- net +9V: track 32.0 -> 0.00 mm
- net Net-(D6-Pad2): track 38.9 -> 69.1 mm
- net inaIN+: track 23.5 -> 52.4 mm
- net Net-(D5-Pad2): track 29.4 -> 56.9 mm
- net Net-(D4-Pad2): track 22.9 -> 44.5 mm
- net Net-(C6-Pad2): track 35.4 -> 54.9 mm
- net bioIN-: track 19.3 -> 0.00 mm
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- added copper zone on B.Cu, net GND
- added copper zone on F.Cu, net GND
Other:
- board size 52.1 x 53.3 mm -> 60.3 x 53.3 mm
- board text added: "A2"
- board text added: "AUDIO OUT"
- board text added: "BATTERY"
- board text added: "C"
- board text added: "D6"
- board text added: "E"
- board text added: "ISOLATED OUTPUT"
- board text added: "LEDs"
- board text added: "S"
- board text added: "SCL"
- board text added: "SDA"
- board text added: "SERVO"
- board text added: "STEMMA ANALOG"
- board text added: "STEMMA DIGITAL"
- board text added: "STEMMA I2C"
- board text added: "VCC"
- board text removed: "AUDIO"
- board text removed: "D2"
- board text removed: "D3"
- board text removed: "D5"
- board text removed: "DIGITAL"
- board text removed: "JAN 2022 - v0.2"
- board text removed: "POWER"
- board text removed: "Upside Down Labs MUSCLE BIOAMP SHIELD"
- board text removed: "https://upsidedownlabs.tech/ MADE IN INDIA"
