File: hardware/Muscle-BioAmpShield.kicad_sch (KiCad schematic)
At the start: 53 parts, among them J1 Audio_output, J2 BioAmp_input, J3 Board_power, J4 Digital_pins, J5 PJ-3062-CO, P1 Power, P2 Analog, P3 Digital, P4 Digital, SW1 SW_Push, SW2 SW_Push, U1 Amp

Commit message: Update to v0.3 KiCad files
Parts:
- removed C12: 100nF, Capacitor_THT:C_Disc_D3.8mm_W2.6mm_P2.50mm, symbol Device:C
- removed J3: Board_power, Connector_JST:JST_PH_S2B-PH-K_1x02_P2.00mm_Horizontal, symbol Connector_Generic:Conn_01x02
- removed J4: Digital_pins, Connector_PinHeader_2.54mm:PinHeader_1x04_P2.54mm_Vertical, symbol Connector_Generic:Conn_01x04
- removed R3, R6: 1K, Resistor_THT:R_Axial_DIN0207_L6.3mm_D2.5mm_P7.62mm_Horizontal, symbol Device:R
- added C11: 100nF, Capacitor_THT:C_Disc_D3.8mm_W2.6mm_P2.50mm, symbol Device:C
- added J10: Servo motor, Connector_PinHeader_2.54mm:PinHeader_1x03_P2.54mm_Vertical, symbol Connector_Generic:Conn_01x03
- added J3: Stemma I2C, Connector_JST:JST_PH_B4B-PH-K_1x04_P2.00mm_Vertical, symbol Connector_Generic:Conn_01x04
- added J4: Stemma Digital D6, Connector_JST:JST_PH_B3B-PH-K_1x03_P2.00mm_Vertical, symbol Connector_Generic:Conn_01x03
- added J6: Isolated Output, Connector_JST:JST_PH_B2B-PH-K_1x02_P2.00mm_Vertical, symbol Connector_Generic:Conn_01x02
- added J7: Stemma Analog A2, Connector_JST:JST_PH_B3B-PH-K_1x03_P2.00mm_Vertical, symbol Connector_Generic:Conn_01x03
- added J8: Stemma I2C, Connector_JST:JST_PH_S4B-PH-K_1x04_P2.00mm_Horizontal, symbol Connector_Generic:Conn_01x04
- added J9: Battery Power, Connector_JST:JST_PH_S2B-PH-K_1x02_P2.00mm_Horizontal, symbol Connector_Generic:Conn_01x02
- added U2: PC817, Package_DIP:DIP-4_W7.62mm, symbol Isolator:PC817
- C1: renamed from C11; value 47uF -> 2.2uF
- C10: value 47uF -> 470uF
- C12: renamed from C6; value 10uF -> 470uF
- C3: renamed from C1; value 1nF -> 100pF
- C5: renamed from C3; value 1nF -> 100pF
- C6: renamed from C8; value 2.2uF -> 1uF
- C8: renamed from C4; value 100nF -> 100pF
- J1: renamed from J2; value BioAmp_input -> BioAmp Input
- R1: renamed from R7; value 1K -> 1M
- R19: renamed from R11; value 15K -> 10K
- R2: renamed from R8; value 1K -> 1M
- R20: renamed from R12; value 15K -> 10K
- R5: renamed from R4; value 10K -> 220K
- R6: renamed from R1; value 1K -> 22K
- R7: renamed from R5; value 1K -> 22K
- R8: renamed from R2; value 10K -> 220K
- renumbered C7 to C2, C2 to C4, C5 to C7, J5 to J2, J1 to J5, R15 to R10, R13 to R11, R16 to R12, R17 to R13, R18 to R14, R19 to R15, R20 to R16, R21 to R17, R22 to R18, R10 to R3, R9 to R4, R14 to R9
Connections:
- net bioIN+ is gone; now on net inaIN+: J1.2 (Pin_2)
- net bioIN- is gone; now on net inaIN-: J1.1 (Pin_1)
- net +5V: now also J10.2 (Pin_2), J3.3 (Pin_3), J4.2 (Pin_2), J7.2 (Pin_2), J8.3 (Pin_3); no longer C8.2
- net +9V: now also C12.1, C11.2, J9.1 (Pin_1)
- net 2: now also J10.1 (Pin_1)
- net 3(**): now also U2.1
- net 6(**): now also J4.1 (Pin_1)
- net A2: now also J7.1 (Pin_1)
- net A4(SDA): now also J3.2 (Pin_2)
- net A5(SCL): now also J3.1 (Pin_1)
- net GND: now also C8.1, C11.1, J10.3 (Pin_3), J3.4 (Pin_4), J4.3 (Pin_3), J7.3 (Pin_3), J8.4 (Pin_4), J9.2 (Pin_2), U2.2
- net ampRef: now also C8.2; no longer C12.1
- net SCL: now reaches P3.1 (Pin_1)
- net SCL: now also J8.1 (Pin_1)
- net SDA: now reaches P3.2 (Pin_2)
- net SDA: now also J8.2 (Pin_2)
- net at C2.2, R1.1, R2.2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: no longer C8.1
- new net: J6.2 (Pin_2), U2.3
- new net: J6.1 (Pin_1), U2.4
Other:
- note added: "Audio output interface"
- note added: "BandPass filter (72Hz - 720Hz)"
- note added: "Battery connector"
- note added: "Instrumentation amplifier (Gain x10)"
- note added: "Isolated Digital Output"
- note added: "Reference Power supply"
- note added: "Servo port"
- note added: "Stemma connectors"
- note removed: "Audio interface"
- note removed: "BandPass filter"
- note removed: "Connectors"
- note removed: "Instrumentation amplifier"
- note removed: "Power supply"
- moved on the sheet: C1, C10, C12, C3, C4, C5, C6, C7, C8, C9, J1, J2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

Commit message: Add prefix DIY
Other:
- title: Muscle BioAmp Shield -> DIY Muscle BioAmp Shield
Changed lines of the file:
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@@
   (paper "A4")
   (title_block
-    (title "Muscle BioAmp Shield")
+    (title "DIY Muscle BioAmp Shield")
     (date "2023-02-13")
     (rev "v0.3")
     (company "Upside Down Labs")
-    (comment 1 "BackYard Brains hardware compatible")
+    (comment 1 "BackYardBrains compatible")
     (comment 2 "Arduino Shield for EMG ")
     (comment 3 "Quad OpAmp based design")
